File: RP2040_Euro_Power.kicad_pcb (KiCad board)
At the start: 2 copper layers, 110 x 110 mm, 158 parts, among them J1 Conn_01x40, J2 Conn_01x40, J3 Power, J4 USB C/USB 2.0, J5 Conn_01x03_Pin, SW1 BOOT, SW2 RESET, U101 TL431A, U2 W25Q128JVS, U4 AMS1117-3.3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

Commit message: Version 2 ready to order
Other:
- board text added: "Loom RP2040 V2 Carson Walls 2/2025"
Changed lines of the file:
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@@
 		)
 	)
-	(gr_text "Loom RP2040 V2\nCarson Walls\n1/2025"
+	(gr_text "Loom RP2040 V2\nCarson Walls\n2/2025"
 		(at 85.307 63.419 0)
 		(layer "F.SilkS")
